File: Hardware/killswitch_84.kicad_pcb (KiCad board)
At the start: 2 copper layers, 25 x 56 mm, 34 parts, among them J1 PWR_IN, J2 REMOTE, J3 PI, Q1 Q_PMOS_GSD, SW1 SW_Push, U1 ATTINY84-20SSU, U2 TSDP341xx, U3 AZ1117-3.3, U4 TXB0108DQSR

Commit message: version bump
Other:
- board text added: "KillSwitch v0.4.11"
- board text removed: "KillSwitch v0.4.10"
Changed lines of the file:
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@@
   (title_block
     (title "KillSwitch on ATTiny84")
-    (date 2019-03-16)
-    (rev 0.4.10)
+    (date 2019-03-17)
+    (rev 0.4.11)
     (company "Dana Hynes")
     (comment 1 "Copyright (c) 2019 ")
@@
     (arrow2b (pts (xy 166.605124 68.993) (xy 167.191545 70.119504)))
   )
-  (gr_text "KillSwitch\nv0.4.10" (at 143.49 77.502) (layer B.SilkS)
+  (gr_text "KillSwitch\nv0.4.11" (at 143.49 77.502) (layer B.SilkS)
     (effects (font (size 1.5 1.5) (thickness 0.3)) (justify mirror))
   )

Commit message: version bump
Other:
- board text added: "KillSwitch v0.4.12"
- board text removed: "KillSwitch v0.4.11"
Changed lines of the file:
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@@
     (title "KillSwitch on ATTiny84")
     (date 2019-03-17)
-    (rev 0.4.11)
+    (rev 0.4.12)
     (company "Dana Hynes")
     (comment 1 "Copyright (c) 2019 ")
@@
     (arrow2b (pts (xy 166.605124 68.993) (xy 167.191545 70.119504)))
   )
-  (gr_text "KillSwitch\nv0.4.11" (at 143.49 77.502) (layer B.SilkS)
+  (gr_text "KillSwitch\nv0.4.12" (at 143.49 77.502) (layer B.SilkS)
     (effects (font (size 1.5 1.5) (thickness 0.3)) (justify mirror))
   )

Commit message: version bump
Other:
- board text added: "KillSwitch v0.4.13"
- board text removed: "KillSwitch v0.4.12"
Changed lines of the file:
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@@
     (title "KillSwitch on ATTiny84")
     (date 2019-03-17)
-    (rev 0.4.12)
+    (rev 0.4.13)
     (company "Dana Hynes")
     (comment 1 "Copyright (c) 2019 ")
@@
     (arrow2b (pts (xy 166.605124 68.993) (xy 167.191545 70.119504)))
   )
-  (gr_text "KillSwitch\nv0.4.12" (at 143.49 77.502) (layer B.SilkS)
+  (gr_text "KillSwitch\nv0.4.13" (at 143.49 77.502) (layer B.SilkS)
     (effects (font (size 1.5 1.5) (thickness 0.3)) (justify mirror))
   )

Commit message: version bump
Other:
- board text added: "KillSwitch v0.4.14"
- board text removed: "KillSwitch v0.4.13"
Changed lines of the file:
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@@
     (title "KillSwitch on ATTiny84")
     (date 2019-03-17)
-    (rev 0.4.13)
+    (rev 0.4.14)
     (company "Dana Hynes")
     (comment 1 "Copyright (c) 2019 ")
@@
     (arrow2b (pts (xy 166.605124 68.993) (xy 167.191545 70.119504)))
   )
-  (gr_text "KillSwitch\nv0.4.13" (at 143.49 77.502) (layer B.SilkS)
+  (gr_text "KillSwitch\nv0.4.14" (at 143.49 77.502) (layer B.SilkS)
     (effects (font (size 1.5 1.5) (thickness 0.3)) (justify mirror))
   )

Commit message: version bump
Other:
- board text added: "KillSwitch v0.4.15"
- board text removed: "KillSwitch v0.4.14"
Changed lines of the file:
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@@
     (title "KillSwitch on ATTiny84")
     (date 2019-03-17)
-    (rev 0.4.14)
+    (rev 0.4.15)
     (company "Dana Hynes")
     (comment 1 "Copyright (c) 2019 ")
@@
     (arrow2b (pts (xy 166.605124 68.993) (xy 167.191545 70.119504)))
   )
-  (gr_text "KillSwitch\nv0.4.14" (at 143.49 77.502) (layer B.SilkS)
+  (gr_text "KillSwitch\nv0.4.15" (at 143.49 77.502) (layer B.SilkS)
     (effects (font (size 1.5 1.5) (thickness 0.3)) (justify mirror))
   )

Commit message: version bump
Other:
- board text added: "KillSwitch v0.4.16"
- board text removed: "KillSwitch v0.4.15"
Changed lines of the file:
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@@
     (title "KillSwitch on ATTiny84")
     (date 2019-03-17)
-    (rev 0.4.15)
+    (rev 0.4.16)
     (company "Dana Hynes")
     (comment 1 "Copyright (c) 2019 ")
@@
     (arrow2b (pts (xy 166.605124 68.993) (xy 167.191545 70.119504)))
   )
-  (gr_text "KillSwitch\nv0.4.15" (at 143.49 77.502) (layer B.SilkS)
+  (gr_text "KillSwitch\nv0.4.16" (at 143.49 77.502) (layer B.SilkS)
     (effects (font (size 1.5 1.5) (thickness 0.3)) (justify mirror))
   )

Commit message: version bump
Other:
- board text added: "KillSwitch v0.4.17"
- board text removed: "KillSwitch v0.4.16"
Changed lines of the file:
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@@
   (title_block
     (title "KillSwitch on ATTiny84")
-    (date 2019-03-17)
-    (rev 0.4.16)
+    (date 2019-03-18)
+    (rev 0.4.17)
     (company "Dana Hynes")
     (comment 1 "Copyright (c) 2019 ")
@@
     (arrow2b (pts (xy 166.605124 68.993) (xy 167.191545 70.119504)))
   )
-  (gr_text "KillSwitch\nv0.4.16" (at 143.49 77.502) (layer B.SilkS)
+  (gr_text "KillSwitch\nv0.4.17" (at 143.49 77.502) (layer B.SilkS)
     (effects (font (size 1.5 1.5) (thickness 0.3)) (justify mirror))
   )

Commit message: fixed typo in setuid
Other:
- board text added: "KillSwitch v0.4.18"
- board text removed: "KillSwitch v0.4.17"
Changed lines of the file:
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@@
     (title "KillSwitch on ATTiny84")
     (date 2019-03-18)
-    (rev 0.4.17)
+    (rev 0.4.18)
     (company "Dana Hynes")
     (comment 1 "Copyright (c) 2019 ")
@@
     (arrow2b (pts (xy 166.605124 68.993) (xy 167.191545 70.119504)))
   )
-  (gr_text "KillSwitch\nv0.4.17" (at 143.49 77.502) (layer B.SilkS)
+  (gr_text "KillSwitch\nv0.4.18" (at 143.49 77.502) (layer B.SilkS)
     (effects (font (size 1.5 1.5) (thickness 0.3)) (justify mirror))
   )
