File: Hardware/Pi3/killswitch-pi3.kicad_pcb (KiCad board)
At the start: 2 copper layers, 25 x 56 mm, 35 parts, among them J1 PWR_IN, J2 REMOTE, J3 PI, Q1 Q_PMOS_GSD, SW1 SW_Push, U1 ATTINY84-20SSU, U2 TSDP341xx, U3 AZ1117-3.3, U4 TXB0108DQSR

Commit message: version bump
Other:
- board text added: "KillSwitch v0.5.8"
- board text removed: "KillSwitch v0.5.7"
Changed lines of the file:
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@@
     (arrow2b (pts (xy 166.605124 68.993) (xy 167.191545 70.119504)))
   )
-  (gr_text "KillSwitch\nv0.5.7" (at 143.49 77.502) (layer B.SilkS)
+  (gr_text "KillSwitch\nv0.5.8" (at 143.49 77.502) (layer B.SilkS)
     (effects (font (size 1.5 1.5) (thickness 0.3)) (justify mirror))
   )

Commit message: version bump
Other:
- board text added: "KillSwitch v0.5.9"
- board text removed: "KillSwitch v0.5.8"
Changed lines of the file:
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@@
     (arrow2b (pts (xy 166.605124 68.993) (xy 167.191545 70.119504)))
   )
-  (gr_text "KillSwitch\nv0.5.8" (at 143.49 77.502) (layer B.SilkS)
+  (gr_text "KillSwitch\nv0.5.9" (at 143.49 77.502) (layer B.SilkS)
     (effects (font (size 1.5 1.5) (thickness 0.3)) (justify mirror))
   )

Commit message: version bump
Other:
- board text added: "KillSwitch v0.5.10"
- board text removed: "KillSwitch v0.5.9"
Changed lines of the file:
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@@
     (arrow2b (pts (xy 166.605124 68.993) (xy 167.191545 70.119504)))
   )
-  (gr_text "KillSwitch\nv0.5.9" (at 143.49 77.502) (layer B.SilkS)
+  (gr_text "KillSwitch\nv0.5.10" (at 143.49 77.502) (layer B.SilkS)
     (effects (font (size 1.5 1.5) (thickness 0.3)) (justify mirror))
   )

Commit message: version bump
Other:
- board text added: "KillSwitch v0.5.12"
- board text removed: "KillSwitch v0.5.10"
Changed lines of the file:
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@@
     (arrow2b (pts (xy 166.605124 68.993) (xy 167.191545 70.119504)))
   )
-  (gr_text "KillSwitch\nv0.5.10" (at 143.49 77.502) (layer B.SilkS)
+  (gr_text "KillSwitch\nv0.5.12" (at 143.49 77.502) (layer B.SilkS)
     (effects (font (size 1.5 1.5) (thickness 0.3)) (justify mirror))
   )

Commit message: version bump
Other:
- board text added: "KillSwitch v0.5.13"
- board text removed: "KillSwitch v0.5.12"
Changed lines of the file:
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@@
     (arrow2b (pts (xy 166.605124 68.993) (xy 167.191545 70.119504)))
   )
-  (gr_text "KillSwitch\nv0.5.12" (at 143.49 77.502) (layer B.SilkS)
+  (gr_text "KillSwitch\nv0.5.13" (at 143.49 77.502) (layer B.SilkS)
     (effects (font (size 1.5 1.5) (thickness 0.3)) (justify mirror))
   )

Commit message: version bump
Other:
- board text added: "KillSwitch v0.5.14"
- board text removed: "KillSwitch v0.5.13"
Changed lines of the file:
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@@
     (arrow2b (pts (xy 166.605124 68.993) (xy 167.191545 70.119504)))
   )
-  (gr_text "KillSwitch\nv0.5.13" (at 143.49 77.502) (layer B.SilkS)
+  (gr_text "KillSwitch\nv0.5.14" (at 143.49 77.502) (layer B.SilkS)
     (effects (font (size 1.5 1.5) (thickness 0.3)) (justify mirror))
   )

Commit message: version bump
Other:
- board text added: "KillSwitch v0.5.15"
- board text removed: "KillSwitch v0.5.14"
Changed lines of the file:
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@@
     (arrow2b (pts (xy 166.605124 68.993) (xy 167.191545 70.119504)))
   )
-  (gr_text "KillSwitch\nv0.5.14" (at 143.49 77.502) (layer B.SilkS)
+  (gr_text "KillSwitch\nv0.5.15" (at 143.49 77.502) (layer B.SilkS)
     (effects (font (size 1.5 1.5) (thickness 0.3)) (justify mirror))
   )

Commit message: version bump
Other:
- board text added: "KillSwitch v0.5.16"
- board text removed: "KillSwitch v0.5.15"
Changed lines of the file:
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@@
     (arrow2b (pts (xy 166.605124 68.993) (xy 167.191545 70.119504)))
   )
-  (gr_text "KillSwitch\nv0.5.15" (at 143.49 77.502) (layer B.SilkS)
+  (gr_text "KillSwitch\nv0.5.16" (at 143.49 77.502) (layer B.SilkS)
     (effects (font (size 1.5 1.5) (thickness 0.3)) (justify mirror))
   )
