File: Hardware/Pi3/killswitch-pi3.kicad_pcb (KiCad board)
At the start: 2 copper layers, 25 x 56 mm, 36 parts, among them J1 PWR_IN, J2 REMOTE, J3 PI, J4 JST, Q1 Q_PMOS_GSD, SW1 SW_Push, U1 ATTINY84-20SSU, U2 TSDP341xx, U3 AZ1117-3.3, U4 TXB0108DQSR

Commit message: first test of retropie
Parts:
- added J5: Conn_01x02, Pin_Headers:Pin_Header_Straight_1x02_Pitch2.54mm, F.Cu at (157.7, 102.6)
- J4: value JST -> Conn_01x02; footprint Connectors_JST:JST_EH_S02B-EH_02x2.50mm_Angled -> Connectors_JST:JST_XH_B02B-XH-A_02x2.50mm_Straight
Routing:
- net GND: track 70.9 -> 66.9 mm
- net +5V: track 126.0 -> 129.8 mm

Commit message: retropie test
Other:
- board text added: "KillSwitch v0.1.4"
- board text removed: "KillSwitch v0.1.0"
Changed lines of the file:
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@@
     (arrow2b (pts (xy 166.605124 68.993) (xy 167.191545 70.119504)))
   )
-  (gr_text "KillSwitch\nv0.1.0" (at 143.49 77.502) (layer B.SilkS)
+  (gr_text "KillSwitch\nv0.1.4" (at 143.49 77.502) (layer B.SilkS)
     (effects (font (size 1.5 1.5) (thickness 0.3)) (justify mirror))
   )

Commit message: retropie test
Other:
- board text added: "KillSwitch v0.1.6"
- board text removed: "KillSwitch v0.1.4"
Changed lines of the file:
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@@
     (arrow2b (pts (xy 166.605124 68.993) (xy 167.191545 70.119504)))
   )
-  (gr_text "KillSwitch\nv0.1.4" (at 143.49 77.502) (layer B.SilkS)
+  (gr_text "KillSwitch\nv0.1.6" (at 143.49 77.502) (layer B.SilkS)
     (effects (font (size 1.5 1.5) (thickness 0.3)) (justify mirror))
   )

Commit message: retropie test
Other:
- board text added: "KillSwitch v0.1.7"
- board text removed: "KillSwitch v0.1.6"
Changed lines of the file:
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@@
     (arrow2b (pts (xy 166.605124 68.993) (xy 167.191545 70.119504)))
   )
-  (gr_text "KillSwitch\nv0.1.6" (at 143.49 77.502) (layer B.SilkS)
+  (gr_text "KillSwitch\nv0.1.7" (at 143.49 77.502) (layer B.SilkS)
     (effects (font (size 1.5 1.5) (thickness 0.3)) (justify mirror))
   )

Commit message: retropie test
Other:
- board text added: "KillSwitch v0.1.8"
- board text removed: "KillSwitch v0.1.7"
Changed lines of the file:
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@@
     (arrow2b (pts (xy 166.605124 68.993) (xy 167.191545 70.119504)))
   )
-  (gr_text "KillSwitch\nv0.1.7" (at 143.49 77.502) (layer B.SilkS)
+  (gr_text "KillSwitch\nv0.1.8" (at 143.49 77.502) (layer B.SilkS)
     (effects (font (size 1.5 1.5) (thickness 0.3)) (justify mirror))
   )

Commit message: retropie test
Other:
- board text added: "KillSwitch v0.1.9"
- board text removed: "KillSwitch v0.1.8"
Changed lines of the file:
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@@
     (arrow2b (pts (xy 166.605124 68.993) (xy 167.191545 70.119504)))
   )
-  (gr_text "KillSwitch\nv0.1.8" (at 143.49 77.502) (layer B.SilkS)
+  (gr_text "KillSwitch\nv0.1.9" (at 143.49 77.502) (layer B.SilkS)
     (effects (font (size 1.5 1.5) (thickness 0.3)) (justify mirror))
   )

Commit message: retropie test
Other:
- board text added: "KillSwitch v0.1.10"
- board text removed: "KillSwitch v0.1.9"
Changed lines of the file:
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@@
     (arrow2b (pts (xy 166.605124 68.993) (xy 167.191545 70.119504)))
   )
-  (gr_text "KillSwitch\nv0.1.9" (at 143.49 77.502) (layer B.SilkS)
+  (gr_text "KillSwitch\nv0.1.10" (at 143.49 77.502) (layer B.SilkS)
     (effects (font (size 1.5 1.5) (thickness 0.3)) (justify mirror))
   )

Commit message: retropie test
Other:
- board text added: "KillSwitch v0.1.11"
- board text removed: "KillSwitch v0.1.10"
Changed lines of the file:
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@@
     (arrow2b (pts (xy 166.605124 68.993) (xy 167.191545 70.119504)))
   )
-  (gr_text "KillSwitch\nv0.1.10" (at 143.49 77.502) (layer B.SilkS)
+  (gr_text "KillSwitch\nv0.1.11" (at 143.49 77.502) (layer B.SilkS)
     (effects (font (size 1.5 1.5) (thickness 0.3)) (justify mirror))
   )
