File: Hardware/Pi3/killswitch-pi3.kicad_pcb (KiCad board)
At the start: 2 copper layers, 25 x 56 mm, 37 parts, among them J1 PWR_IN, J2 REMOTE, J3 PI, J4 Conn_01x02, J5 Conn_01x02, Q1 Q_PMOS_GSD, SW1 SW_Push, U1 ATTINY84-20SSU, U2 TSDP341xx, U3 AZ1117-3.3, U4 TXB0108DQSR

Commit message: retropie test
Other:
- board text added: "KillSwitch v0.1.12"
- board text removed: "KillSwitch v0.1.11"
Changed lines of the file:
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@@
     (arrow2b (pts (xy 166.605124 68.993) (xy 167.191545 70.119504)))
   )
-  (gr_text "KillSwitch\nv0.1.11" (at 143.49 77.502) (layer B.SilkS)
+  (gr_text "KillSwitch\nv0.1.12" (at 143.49 77.502) (layer B.SilkS)
     (effects (font (size 1.5 1.5) (thickness 0.3)) (justify mirror))
   )

Commit message: retropie test
Other:
- board text added: "KillSwitch v0.1.13"
- board text removed: "KillSwitch v0.1.12"
Changed lines of the file:
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@@
     (arrow2b (pts (xy 166.605124 68.993) (xy 167.191545 70.119504)))
   )
-  (gr_text "KillSwitch\nv0.1.12" (at 143.49 77.502) (layer B.SilkS)
+  (gr_text "KillSwitch\nv0.1.13" (at 143.49 77.502) (layer B.SilkS)
     (effects (font (size 1.5 1.5) (thickness 0.3)) (justify mirror))
   )

Commit message: retropie test
Other:
- board text added: "KillSwitch v0.1.15"
- board text removed: "KillSwitch v0.1.13"
Changed lines of the file:
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@@
     (arrow2b (pts (xy 166.605124 68.993) (xy 167.191545 70.119504)))
   )
-  (gr_text "KillSwitch\nv0.1.13" (at 143.49 77.502) (layer B.SilkS)
+  (gr_text "KillSwitch\nv0.1.15" (at 143.49 77.502) (layer B.SilkS)
     (effects (font (size 1.5 1.5) (thickness 0.3)) (justify mirror))
   )

Commit message: install-latest.sh test
Other:
- board text added: "KillSwitch v0.1.16"
- board text removed: "KillSwitch v0.1.15"
Changed lines of the file:
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@@
     (arrow2b (pts (xy 166.605124 68.993) (xy 167.191545 70.119504)))
   )
-  (gr_text "KillSwitch\nv0.1.15" (at 143.49 77.502) (layer B.SilkS)
+  (gr_text "KillSwitch\nv0.1.16" (at 143.49 77.502) (layer B.SilkS)
     (effects (font (size 1.5 1.5) (thickness 0.3)) (justify mirror))
   )

Commit message: test
Other:
- board text added: "KillSwitch v0.1.17"
- board text removed: "KillSwitch v0.1.16"
Changed lines of the file:
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@@
     (arrow2b (pts (xy 166.605124 68.993) (xy 167.191545 70.119504)))
   )
-  (gr_text "KillSwitch\nv0.1.16" (at 143.49 77.502) (layer B.SilkS)
+  (gr_text "KillSwitch\nv0.1.17" (at 143.49 77.502) (layer B.SilkS)
     (effects (font (size 1.5 1.5) (thickness 0.3)) (justify mirror))
   )

Commit message: test
Other:
- board text added: "KillSwitch v0.1.18"
- board text removed: "KillSwitch v0.1.17"
Changed lines of the file:
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@@
     (arrow2b (pts (xy 166.605124 68.993) (xy 167.191545 70.119504)))
   )
-  (gr_text "KillSwitch\nv0.1.17" (at 143.49 77.502) (layer B.SilkS)
+  (gr_text "KillSwitch\nv0.1.18" (at 143.49 77.502) (layer B.SilkS)
     (effects (font (size 1.5 1.5) (thickness 0.3)) (justify mirror))
   )

Commit message: test
Other:
- board text added: "KillSwitch v0.1.19"
- board text removed: "KillSwitch v0.1.18"
Changed lines of the file:
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@@
     (arrow2b (pts (xy 166.605124 68.993) (xy 167.191545 70.119504)))
   )
-  (gr_text "KillSwitch\nv0.1.18" (at 143.49 77.502) (layer B.SilkS)
+  (gr_text "KillSwitch\nv0.1.19" (at 143.49 77.502) (layer B.SilkS)
     (effects (font (size 1.5 1.5) (thickness 0.3)) (justify mirror))
   )

Commit message: test
Other:
- board text added: "KillSwitch v0.1.20"
- board text removed: "KillSwitch v0.1.19"
Changed lines of the file:
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@@
     (arrow2b (pts (xy 166.605124 68.993) (xy 167.191545 70.119504)))
   )
-  (gr_text "KillSwitch\nv0.1.19" (at 143.49 77.502) (layer B.SilkS)
+  (gr_text "KillSwitch\nv0.1.20" (at 143.49 77.502) (layer B.SilkS)
     (effects (font (size 1.5 1.5) (thickness 0.3)) (justify mirror))
   )
