File: Hardware/Pi3/killswitch-pi3.sch (KiCad schematic (older format))
At the start: 30 parts, among them J1 PWR_IN, J2 REMOTE, J3 PI, Q1 Q_PMOS_GSD, SW1 SW_Push, U1 ATTINY84-20SSU, U2 TSDP341xx, U3 AZ1117-3.3, U4 TXB0108DQSR

Commit message: first public release
Parts:
- added J4: JST, Connectors_JST:JST_EH_S02B-EH_02x2.50mm_Angled, symbol conn:Conn_01x02_Female
Connections:
- net +5V: now also J4.1 (Pin_1)
- net GND: now also J4.2 (Pin_2)
Changed lines of the file:
@@
 Wire Wire Line
 	4000 2700 6300 2700
+$Comp
+L conn:Conn_01x02_Female J4
+U 1 1 5CDDD424
+P 1100 4050
+F 0 "J4" V 1040 3862 50  0000 R CNN
+F 1 "JST" V 949 3862 50  0000 R CNN
+F 2 "Connectors_JST:JST_EH_S02B-EH_02x2.50mm_Angled" H 1100 4050 50  0001 C CNN
+F 3 "~" H 1100 4050 50  0001 C CNN
+	1    1100 4050
+	0    -1   -1   0
+$EndComp
+$Comp
+L power:+5V #PWR0102
+U 1 1 5CDE9ACD
+P 1100 4450
+F 0 "#PWR0102" H 1100 4300 50  0001 C CNN
+F 1 "+5V" H 1115 4623 50  0000 C CNN
+F 2 "" H 1100 4450 50  0001 C CNN
+F 3 "" H 1100 4450 50  0001 C CNN
+	1    1100 4450
+	-1   0    0    1
+$EndComp
+$Comp
+L power:GND #PWR0103
+U 1 1 5CDE9B91
+P 1200 4450
+F 0 "#PWR0103" H 1200 4200 50  0001 C CNN
+F 1 "GND" H 1205 4277 50  0000 C CNN
+F 2 "" H 1200 4450 50  0001 C CNN
+F 3 "" H 1200 4450 50  0001 C CNN
+	1    1200 4450
+	1    0    0    -1
+$EndComp
+Wire Wire Line
+	1200 4450 1200 4250
+Wire Wire Line
+	1100 4250 1100 4450
 $EndSCHEMATC

Commit message: first test of retropie
Parts:
- removed J4: JST, Connectors_JST:JST_EH_S02B-EH_02x2.50mm_Angled, symbol conn:Conn_01x02_Female
- added J4: Conn_01x02, Connectors_JST:JST_XH_B02B-XH-A_02x2.50mm_Straight, symbol conn:Conn_01x02
- added J5: Conn_01x02, Pin_Headers:Pin_Header_Straight_1x02_Pitch2.54mm, symbol conn:Conn_01x02
Connections:
- net +5V: now also J4.1 (Pin_1), J5.1 (Pin_1)
- net GND: now also J4.2 (Pin_2), J5.2 (Pin_2)
Changed lines of the file:
@@
 	4000 2700 6300 2700
-$Comp
-L conn:Conn_01x02_Female J4
-U 1 1 5CDDD424
-P 1100 4050
-F 0 "J4" V 1040 3862 50  0000 R CNN
-F 1 "JST" V 949 3862 50  0000 R CNN
-F 2 "Connectors_JST:JST_EH_S02B-EH_02x2.50mm_Angled" H 1100 4050 50  0001 C CNN
-F 3 "~" H 1100 4050 50  0001 C CNN
-	1    1100 4050
-	0    -1   -1   0
-$EndComp
 $Comp
 L power:+5V #PWR0102
@@
 Wire Wire Line
 	1100 4250 1100 4450
+$Comp
+L conn:Conn_01x02 J5
+U 1 1 5CDF1F59
+P 1100 4850
+F 0 "J5" V 1066 4662 50  0000 R CNN
+F 1 "Conn_01x02" V 975 4662 50  0000 R CNN
+F 2 "Pin_Headers:Pin_Header_Straight_1x02_Pitch2.54mm" H 1100 4850 50  0001 C CNN
+F 3 "~" H 1100 4850 50  0001 C CNN
+	1    1100 4850
+	0    -1   -1   0
+$EndComp
+$Comp
+L conn:Conn_01x02 J4
+U 1 1 5CDF20BC
+P 1100 4050
+F 0 "J4" V 1066 3862 50  0000 R CNN
+F 1 "Conn_01x02" V 975 3862 50  0000 R CNN
+F 2 "Connectors_JST:JST_XH_B02B-XH-A_02x2.50mm_Straight" H 1100 4050 50  0001 C CNN
+F 3 "~" H 1100 4050 50  0001 C CNN
+	1    1100 4050
+	0    -1   -1   0
+$EndComp
+$Comp
+L power:+5V #PWR026
+U 1 1 5CDF21A0
+P 1100 5250
+F 0 "#PWR026" H 1100 5100 50  0001 C CNN
+F 1 "+5V" H 1115 5423 50  0000 C CNN
+F 2 "" H 1100 5250 50  0001 C CNN
+F 3 "" H 1100 5250 50  0001 C CNN
+	1    1100 5250
+	-1   0    0    1
+$EndComp
+$Comp
+L power:GND #PWR027
+U 1 1 5CDF21A6
+P 1200 5250
+F 0 "#PWR027" H 1200 5000 50  0001 C CNN
+F 1 "GND" H 1205 5077 50  0000 C CNN
+F 2 "" H 1200 5250 50  0001 C CNN
+F 3 "" H 1200 5250 50  0001 C CNN
+	1    1200 5250
+	1    0    0    -1
+$EndComp
+Wire Wire Line
+	1200 5250 1200 5050
+Wire Wire Line
+	1100 5050 1100 5250
 $EndSCHEMATC
