File: Hardware/Pi0/killswitch-pi0.kicad_pcb (KiCad board)
At the start: 2 copper layers, 65 x 30 mm, 35 parts, among them J2 REMOTE, J3 PI, Q1 Q_PMOS_GSD, SW1 SW_Push, U1 ATTINY84-20SSU, U2 TSDP341xx, U3 AZ1117-3.3, U4 TXB0108DQSR

Commit message: version bump
Other:
- board text added: "KillSwitch v0.5.18"
- board text removed: "KillSwitch v0.5.17"
Changed lines of the file:
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@@
     (title "KillSwitch for Pi Zero")
     (date "2019-05-03")
-    (rev "0.5.17")
+    (rev "0.5.18")
   )
   (layers
@@
     (effects (font (size 0.8 0.8) (thickness 0.1)))
   )
-  (gr_text "KillSwitch\nv0.5.17" (at 91.152 99.03 90) (layer B.SilkS)
+  (gr_text "KillSwitch\nv0.5.18" (at 91.152 99.03 90) (layer B.SilkS)
     (effects (font (size 1.5 1.5) (thickness 0.3)) (justify mirror))
   )

Commit message: version bump
Other:
- board text added: "KillSwitch v0.5.19"
- board text removed: "KillSwitch v0.5.18"
Changed lines of the file:
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@@
   (title_block
     (title "KillSwitch for Pi Zero")
-    (date "2019-05-03")
-    (rev "0.5.18")
+    (date "2019-05-07")
+    (rev "0.5.19")
   )
   (layers
@@
     (effects (font (size 0.8 0.8) (thickness 0.1)))
   )
-  (gr_text "KillSwitch\nv0.5.18" (at 91.152 99.03 90) (layer B.SilkS)
+  (gr_text "KillSwitch\nv0.5.19" (at 91.152 99.03 90) (layer B.SilkS)
     (effects (font (size 1.5 1.5) (thickness 0.3)) (justify mirror))
   )

Commit message: version bump
Other:
- board text added: "KillSwitch v0.5.20"
- board text removed: "KillSwitch v0.5.19"
Changed lines of the file:
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@@
   (title_block
     (title "KillSwitch for Pi Zero")
-    (date "2019-05-07")
-    (rev "0.5.19")
+    (date "2019-05-08")
+    (rev "0.5.20")
   )
   (layers
@@
     (effects (font (size 0.8 0.8) (thickness 0.1)))
   )
-  (gr_text "KillSwitch\nv0.5.19" (at 91.152 99.03 90) (layer B.SilkS)
+  (gr_text "KillSwitch\nv0.5.20" (at 91.152 99.03 90) (layer B.SilkS)
     (effects (font (size 1.5 1.5) (thickness 0.3)) (justify mirror))
   )

Commit message: version bump for update test
Other:
- board text added: "KillSwitch v0.5.21"
- board text removed: "KillSwitch v0.5.20"
Changed lines of the file:
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@@
   (title_block
     (title "KillSwitch for Pi Zero")
-    (date "2019-05-08")
-    (rev "0.5.20")
+    (date "2019-05-10")
+    (rev "0.5.21")
   )
   (layers
@@
     (effects (font (size 0.8 0.8) (thickness 0.1)))
   )
-  (gr_text "KillSwitch\nv0.5.20" (at 91.152 99.03 90) (layer B.SilkS)
+  (gr_text "KillSwitch\nv0.5.21" (at 91.152 99.03 90) (layer B.SilkS)
     (effects (font (size 1.5 1.5) (thickness 0.3)) (justify mirror))
   )

Commit message: first public release
Other:
- board text added: "KillSwitch v0.1.0"
- board text removed: "KillSwitch v0.5.21"
Changed lines of the file:
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@@
   (title_block
     (title "KillSwitch for Pi Zero")
-    (date "2019-05-10")
-    (rev "0.5.21")
+    (date "2019-05-14")
+    (rev "0.1.0")
   )
   (layers
@@
     (effects (font (size 0.8 0.8) (thickness 0.1)))
   )
-  (gr_text "KillSwitch\nv0.5.21" (at 91.152 99.03 90) (layer B.SilkS)
+  (gr_text "KillSwitch\nv0.1.0" (at 91.152 99.03 90) (layer B.SilkS)
     (effects (font (size 1.5 1.5) (thickness 0.3)) (justify mirror))
   )

Commit message: minor edits
Other:
- board text added: "KillSwitch v0.1.1"
- board text removed: "KillSwitch v0.1.0"
Changed lines of the file:
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@@
     (title "KillSwitch for Pi Zero")
     (date "2019-05-14")
-    (rev "0.1.0")
+    (rev "0.1.1")
   )
   (layers
@@
     (effects (font (size 0.8 0.8) (thickness 0.1)))
   )
-  (gr_text "KillSwitch\nv0.1.0" (at 91.152 99.03 90) (layer B.SilkS)
+  (gr_text "KillSwitch\nv0.1.1" (at 91.152 99.03 90) (layer B.SilkS)
     (effects (font (size 1.5 1.5) (thickness 0.3)) (justify mirror))
   )

Commit message: first public release
Other:
- board text added: "KillSwitch v0.1.0"
- board text removed: "KillSwitch v0.1.1"
Changed lines of the file:
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@@
   (title_block
     (title "KillSwitch for Pi Zero")
-    (date "2019-05-14")
-    (rev "0.1.1")
+    (date "2019-05-16")
+    (rev "0.1.0")
   )
   (layers
@@
     (effects (font (size 0.8 0.8) (thickness 0.1)))
   )
-  (gr_text "KillSwitch\nv0.1.1" (at 91.152 99.03 90) (layer B.SilkS)
+  (gr_text "KillSwitch\nv0.1.0" (at 91.152 99.03 90) (layer B.SilkS)
     (effects (font (size 1.5 1.5) (thickness 0.3)) (justify mirror))
   )

Commit message: retropie test
Other:
- board text added: "KillSwitch v0.1.4"
- board text removed: "KillSwitch v0.1.0"
Changed lines of the file:
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@@
   (title_block
     (title "KillSwitch for Pi Zero")
-    (date "2019-05-16")
-    (rev "0.1.0")
+    (date "2019-05-23")
+    (rev "0.1.4")
   )
   (layers
@@
     (effects (font (size 0.8 0.8) (thickness 0.1)))
   )
-  (gr_text "KillSwitch\nv0.1.0" (at 91.152 99.03 90) (layer B.SilkS)
+  (gr_text "KillSwitch\nv0.1.4" (at 91.152 99.03 90) (layer B.SilkS)
     (effects (font (size 1.5 1.5) (thickness 0.3)) (justify mirror))
   )
