File: Hardware/Pi0/killswitch-pi0.kicad_pcb (KiCad board)
At the start: 2 copper layers, 65 x 30 mm, 35 parts, among them J2 REMOTE, J3 PI, Q1 Q_PMOS_GSD, SW1 SW_Push, U1 ATTINY84-20SSU, U2 TSDP341xx, U3 AZ1117-3.3, U4 TXB0108DQSR

Commit message: test
Other:
- board text added: "KillSwitch v0.1.33"
- board text removed: "KillSwitch v0.1.32"
Changed lines of the file:
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@@
     (title "KillSwitch for Pi Zero")
     (date "2019-06-11")
-    (rev "0.1.32")
+    (rev "0.1.33")
   )
   (layers
@@
     (effects (font (size 0.8 0.8) (thickness 0.1)))
   )
-  (gr_text "KillSwitch\nv0.1.32" (at 91.152 99.03 90) (layer B.SilkS)
+  (gr_text "KillSwitch\nv0.1.33" (at 91.152 99.03 90) (layer B.SilkS)
     (effects (font (size 1.5 1.5) (thickness 0.3)) (justify mirror))
   )

Commit message: test
Other:
- board text added: "KillSwitch v0.1.34"
- board text removed: "KillSwitch v0.1.33"
Changed lines of the file:
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@@
     (title "KillSwitch for Pi Zero")
     (date "2019-06-11")
-    (rev "0.1.33")
+    (rev "0.1.34")
   )
   (layers
@@
     (effects (font (size 0.8 0.8) (thickness 0.1)))
   )
-  (gr_text "KillSwitch\nv0.1.33" (at 91.152 99.03 90) (layer B.SilkS)
+  (gr_text "KillSwitch\nv0.1.34" (at 91.152 99.03 90) (layer B.SilkS)
     (effects (font (size 1.5 1.5) (thickness 0.3)) (justify mirror))
   )

Commit message: test
Other:
- board text added: "KillSwitch v0.1.36"
- board text removed: "KillSwitch v0.1.34"
Changed lines of the file:
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@@
     (title "KillSwitch for Pi Zero")
     (date "2019-06-11")
-    (rev "0.1.34")
+    (rev "0.1.36")
   )
   (layers
@@
     (effects (font (size 0.8 0.8) (thickness 0.1)))
   )
-  (gr_text "KillSwitch\nv0.1.34" (at 91.152 99.03 90) (layer B.SilkS)
+  (gr_text "KillSwitch\nv0.1.36" (at 91.152 99.03 90) (layer B.SilkS)
     (effects (font (size 1.5 1.5) (thickness 0.3)) (justify mirror))
   )

Commit message: test
Other:
- board text added: "KillSwitch v0.1.37"
- board text removed: "KillSwitch v0.1.36"
Changed lines of the file:
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@@
   (title_block
     (title "KillSwitch for Pi Zero")
-    (date "2019-06-11")
-    (rev "0.1.36")
+    (date "2019-06-12")
+    (rev "0.1.37")
   )
   (layers
@@
     (effects (font (size 0.8 0.8) (thickness 0.1)))
   )
-  (gr_text "KillSwitch\nv0.1.36" (at 91.152 99.03 90) (layer B.SilkS)
+  (gr_text "KillSwitch\nv0.1.37" (at 91.152 99.03 90) (layer B.SilkS)
     (effects (font (size 1.5 1.5) (thickness 0.3)) (justify mirror))
   )

Commit message: test
Other:
- board text added: "KillSwitch v0.1.38"
- board text removed: "KillSwitch v0.1.37"
Changed lines of the file:
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@@
     (title "KillSwitch for Pi Zero")
     (date "2019-06-12")
-    (rev "0.1.37")
+    (rev "0.1.38")
   )
   (layers
@@
     (effects (font (size 0.8 0.8) (thickness 0.1)))
   )
-  (gr_text "KillSwitch\nv0.1.37" (at 91.152 99.03 90) (layer B.SilkS)
+  (gr_text "KillSwitch\nv0.1.38" (at 91.152 99.03 90) (layer B.SilkS)
     (effects (font (size 1.5 1.5) (thickness 0.3)) (justify mirror))
   )

Commit message: test
Other:
- board text added: "KillSwitch v0.1.39"
- board text removed: "KillSwitch v0.1.38"
Changed lines of the file:
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@@
     (title "KillSwitch for Pi Zero")
     (date "2019-06-12")
-    (rev "0.1.38")
+    (rev "0.1.39")
   )
   (layers
@@
     (effects (font (size 0.8 0.8) (thickness 0.1)))
   )
-  (gr_text "KillSwitch\nv0.1.38" (at 91.152 99.03 90) (layer B.SilkS)
+  (gr_text "KillSwitch\nv0.1.39" (at 91.152 99.03 90) (layer B.SilkS)
     (effects (font (size 1.5 1.5) (thickness 0.3)) (justify mirror))
   )

Commit message: test
Other:
- board text added: "KillSwitch v0.1.40"
- board text removed: "KillSwitch v0.1.39"
Changed lines of the file:
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@@
     (title "KillSwitch for Pi Zero")
     (date "2019-06-12")
-    (rev "0.1.39")
+    (rev "0.1.40")
   )
   (layers
@@
     (effects (font (size 0.8 0.8) (thickness 0.1)))
   )
-  (gr_text "KillSwitch\nv0.1.39" (at 91.152 99.03 90) (layer B.SilkS)
+  (gr_text "KillSwitch\nv0.1.40" (at 91.152 99.03 90) (layer B.SilkS)
     (effects (font (size 1.5 1.5) (thickness 0.3)) (justify mirror))
   )

Commit message: test
Other:
- board text added: "KillSwitch v0.1.41"
- board text removed: "KillSwitch v0.1.40"
Changed lines of the file:
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@@
     (title "KillSwitch for Pi Zero")
     (date "2019-06-12")
-    (rev "0.1.40")
+    (rev "0.1.41")
   )
   (layers
@@
     (effects (font (size 0.8 0.8) (thickness 0.1)))
   )
-  (gr_text "KillSwitch\nv0.1.40" (at 91.152 99.03 90) (layer B.SilkS)
+  (gr_text "KillSwitch\nv0.1.41" (at 91.152 99.03 90) (layer B.SilkS)
     (effects (font (size 1.5 1.5) (thickness 0.3)) (justify mirror))
   )
